File: Hardware/Qwiic_Button.brd (EAGLE design)
At the start: 25.4 x 25.4 mm, 48 parts, among them J2 QWIIC_RIGHT_ANGLE, J3 QWIIC_RIGHT_ANGLE, J7 ISP, U4 ATTINY84-ARDUINO

Commit message: post design review changes
Parts:
- LOGO3: value SFE_LOGO_NAME_FLAME.1_INCH -> SFE_LOGO_NAME.1_INCH; device SparkFun-Aesthetics:SFE_LOGO_NAME_FLAME_.1 -> SparkFun-Aesthetics:SFE_LOGO_NAME_.1
- moved JP6 7.65 mm to (1.27, 8.26)
- moved JP8 7.65 mm to (1.27, 8.26)
- moved J1 7.62 mm to (15.2, 1.27), turned to 180 degrees
- moved U$5 7.62 mm to (15.2, 1.65)
- moved U$8 7.62 mm to (7.62, 1.65)
- moved LOGO3 7.24 mm to (12.8, 21.2)
- moved J7 2.54 mm to (12.7, 17.8), turned to 90 degrees
- moved U$6 2.54 mm to (12.7, 1.65)
- moved U$7 2.54 mm to (10.2, 1.65)
- moved U$3 0.19 mm to (1.27, 7.30)
Routing:
- net MISO: track 20.9 -> 14.8 mm, vias 2 -> 1
- net 3.3V: track 64.5 -> 60.3 mm, vias 2 -> 3
- net !RST: track 21.0 -> 24.0 mm
- net SDA: track 48.9 -> 48.0 mm, vias 5 -> 6
- net SCL: track 49.3 -> 48.4 mm, vias 3 -> 7
Other:
- board text added: "Fisher M."
- board text added: "v10"
- board text removed: "Priyanka Makin"
- board text removed: "v01"
